File: Electronics V3/LasaurDriverBoard2.brd (EAGLE design)
At the start: 100 x 100 mm, 126 parts, among them IC1 ATMEGA168-20P, IC2 ATMEGA168-20P, IC6 MCP2200SOIC20, Q8 12Mhz, X1 22-23-2021, X3 USB-SMD-NS, Y1 16Mhz, Y2 16Mhz

Commit message: Minor Updates
Minor Updates
Parts:
- removed FCH, FD1, FD2: (no value), led:LED3MM
- removed R31, R32, R33: (no value), resistor:M1206
Connections:
- removed net N$25: FD1.A, R31.1
- removed net N$26: FD2.A, R32.1
- removed net N$27: FCH.A, R33.1
- net CHILLER_BIT_SENSE: no longer FCH.K
- net DOOR1: no longer FD1.K
- net DOOR2: no longer FD2.K
- net VCC: no longer R31.2, R32.2, R33.2
Routing:
- net VCC: track 535.7 -> 526.5 mm
- net N$27: track 5.34 -> 0.00 mm
- net DOOR2: track 76.1 -> 71.8 mm
- net N$26: track 3.68 -> 0.00 mm
- net N$25: track 3.58 -> 0.00 mm
- net DOOR1: track 60.3 -> 57.9 mm
Changed lines of the file:
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@@
 <element name="FZP" library="led" package="LED3MM" value="" x="17.904525" y="66.231315625" rot="R90"/>
 <element name="R30" library="resistor" package="M1206" value="" x="18.857025" y="61.786315625"/>
-<element name="FD1" library="led" package="LED3MM" value="" x="17.904525" y="76.391315625" rot="R90"/>
-<element name="R31" library="resistor" package="M1206" value="" x="18.857025" y="71.628815625"/>
-<element name="FD2" library="led" package="LED3MM" value="" x="17.904525" y="86.868815625" rot="R90"/>
-<element name="R32" library="resistor" package="M1206" value="" x="18.857025" y="82.106315625"/>
-<element name="FCH" library="led" package="LED3MM" value="" x="94.559203125" y="60.24530625" rot="R270"/>
-<element name="R33" library="resistor" package="M1206" value="" x="94.63653125" y="66.176840625" rot="R90"/>
 <element name="ZSTEP" library="con-wago-500" package="W237-102" value="" x="37.797865625" y="97.26631875">
 <attribute name="OC_NEWARK" value="70K9898" x="37.797865625" y="97.26631875" size="1.778" layer="27" display="off"/>
@@
 <contactref element="V2" pad="10"/>
 <contactref element="R20" pad="2"/>
-<contactref element="FCH" pad="K"/>
 <contactref element="CHILLER" pad="2"/>
 <contactref element="R3" pad="1"/>
@@
 <wire x1="96.821175" y1="58.32015625" x2="96.38479375" y2="58.7565375" width="0.8128" layer="1"/>
 <wire x1="96.38479375" y1="58.7565375" x2="94.777971875" y2="58.7565375" width="0.8128" layer="1"/>
-<wire x1="94.777971875" y1="58.7565375" x2="94.559203125" y2="58.97530625" width="0.8128" layer="1"/>
 <wire x1="90.584075" y1="54.929709375" x2="91.681515625" y2="54.929709375" width="0.8128" layer="1"/>
 <wire x1="91.681515625" y1="54.929709375" x2="93.976509375" y2="52.634715625" width="0.8128" layer="1"/>
@@
 <contactref element="R29" pad="2"/>
 <contactref element="R30" pad="2"/>
-<contactref element="R31" pad="2"/>
-<contactref element="R32" pad="2"/>
-<contactref element="R33" pad="2"/>
 <wire x1="14.4487125" y1="18.253503125" x2="15.9642125" y2="18.253503125" width="0.8128" layer="1"/>
 <wire x1="15.9642125" y1="18.253503125" x2="16.634525" y2="18.923815625" width="0.8128" layer="1"/>
@@
 <wire x1="20.444525" y1="69.723815625" x2="20.444525" y2="70.358815625" width="0.8128" layer="1"/>
 <wire x1="20.444525" y1="70.358815625" x2="20.444525" y2="71.441315625" width="0.8128" layer="1"/>
-<wire x1="20.444525" y1="71.441315625" x2="20.257025" y2="71.628815625" width="0.8128" layer="1"/>
 <wire x1="19.809525" y1="18.923815625" x2="20.444525" y2="18.923815625" width="0.8128" layer="1"/>
 <wire x1="20.444525" y1="18.923815625" x2="21.079525" y2="18.288815625" width="0.8128" layer="1"/>
@@
 <wire x1="20.762025" y1="64.961315625" x2="20.762025" y2="70.993815625" width="0.8128" layer="1"/>
 <wire x1="20.762025" y1="70.993815625" x2="20.444525" y2="70.358815625" width="0.8128" layer="1"/>
-<wire x1="20.257025" y1="71.628815625" x2="20.257025" y2="72.076315625" width="0.8128" layer="1"/>
 <wire x1="20.257025" y1="72.076315625" x2="20.762025" y2="72.898815625" width="0.8128" layer="1"/>
 <wire x1="20.762025" y1="72.898815625" x2="20.762025" y2="79.566315625" width="0.8128" layer="1"/>
 <wire x1="20.762025" y1="79.566315625" x2="20.762025" y2="81.283815625" width="0.8128" layer="1"/>
 <wire x1="20.762025" y1="81.283815625" x2="20.67841875" y2="81.419984375" width="0.8128" layer="1"/>
-<wire x1="20.67841875" y1="81.419984375" x2="20.257025" y2="82.106315625" width="0.8128" layer="1"/>
 <wire x1="5.839525" y1="73.891315625" x2="12.467025" y2="73.891315625" width="0.8128" layer="1"/>
 <wire x1="12.467025" y1="73.891315625" x2="14.729525" y2="71.628815625" width="0.8128" layer="1"/>
@@
 <wire x1="57.6618" y1="55.32144375" x2="66.622" y2="55.32144375" width="0.8128" layer="16"/>
 <wire x1="66.622" y1="55.32144375" x2="67.4948" y2="54.44864375" width="0.8128" layer="16"/>
-<wire x1="94.63653125" y1="67.576840625" x2="87.00508125" y2="67.576840625" width="0.8128" layer="1"/>
 <wire x1="87.00508125" y1="67.576840625" x2="86.959390625" y2="67.62253125" width="0.8128" layer="1"/>
 <wire x1="27.17699375" y1="26.242221875" x2="27.17699375" y2="24.91861875" width="0.8128" layer="1"/>
@@
 <vertex x="0.442025" y="-2.031184375"/>
 </polygon>
+<wire x1="97.797928125" y1="34.353253125" x2="95.574315625" y2="34.353253125" width="0" layer="19" extent="16-16"/>
+<wire x1="20.257025" y1="72.076315625" x2="20.444525" y2="71.441315625" width="0" layer="19" extent="1-1"/>
 </signal>
 <signal name="MCRTS">
@@
 <contactref element="R18" pad="2"/>
 <contactref element="DOOR1" pad="2"/>
-<contactref element="FD1" pad="K"/>
 <wire x1="5.839525" y1="78.891315625" x2="11.554525" y2="78.891315625" width="0.8128" layer="1"/>
 <wire x1="11.554525" y1="78.891315625" x2="17.309525" y2="78.891315625" width="0.8128" layer="1"/>
-<wire x1="17.309525" y1="78.891315625" x2="17.904525" y2="77.661315625" width="0.8128" layer="1"/>
 <wire x1="25.38053125" y1="41.340265625" x2="23.745575" y2="41.340265625" width="0.4064" layer="1"/>
 <wire x1="23.745575" y1="41.340265625" x2="22.984525" y2="42.101315625" width="0.4064" layer="1"/>
@@
 <via x="24.254525" y="77.343815625" extent="1-16" drill="0.6" shape="square"/>
 <wire x1="24.254525" y1="77.343815625" x2="18.857025" y2="77.343815625" width="0.4064" layer="16"/>
-<wire x1="18.857025" y1="77.343815625" x2="17.904525" y2="77.661315625" width="0.4064" layer="16"/>
 <wire x1="11.742025" y1="76.391315625" x2="11.742025" y2="78.703815625" width="0.6096" layer="1"/>
 <wire x1="11.742025" y1="78.703815625" x2="11.554525" y2="78.891315625" width="0.6096" layer="1"/>
+<wire x1="18.857025" y1="77.343815625" x2="17.309525" y2="78.891315625" width="0" layer="19" extent="1-16"/>
 </signal>
 <signal name="DOOR2">
@@
 <contactref element="R15" pad="2"/>
 <contactref element="DOOR2" pad="2"/>
-<contactref element="FD2" pad="K"/>
 <wire x1="5.839525" y1="89.051315625" x2="17.309525" y2="89.051315625" width="0.8128" layer="1"/>
-<wire x1="17.309525" y1="89.051315625" x2="17.904525" y2="88.138815625" width="0.8128" layer="1"/>
 <wire x1="25.38053125" y1="38.800265625" x2="23.110575" y2="38.800265625" width="0.4064" layer="1"/>
 <wire x1="23.110575" y1="38.800265625" x2="22.032025" y2="39.878815625" width="0.4064" layer="1"/>
 <wire x1="22.032025" y1="39.878815625" x2="22.032025" y2="86.868815625" width="0.4064" layer="1"/>
 <wire x1="22.032025" y1="86.868815625" x2="21.079525" y2="88.138815625" width="0.4064" layer="1"/>
-<wire x1="21.079525" y1="88.138815625" x2="17.904525" y2="88.138815625" width="0.4064" layer="1"/>
 <wire x1="5.839525" y1="89.051315625" x2="10.959525" y2="89.051315625" width="0.6096" layer="1"/>
 <wire x1="10.959525" y1="89.051315625" x2="11.554525" y2="88.456315625" width="0.6096" layer="1"/>
 <wire x1="11.554525" y1="88.456315625" x2="11.554525" y2="86.738815625" width="0.6096" layer="1"/>
 <wire x1="11.554525" y1="86.738815625" x2="11.742025" y2="86.551315625" width="0.6096" layer="1"/>
+<wire x1="21.079525" y1="88.138815625" x2="17.309525" y2="89.051315625" width="0" layer="19" extent="1-1"/>
 </signal>
 <signal name="LASER_PROT">
@@
 <wire x1="17.457025" y1="64.196315625" x2="17.904525" y2="64.961315625" width="0.8128" layer="1"/>
 </signal>
-<signal name="N$25">
-<contactref element="FD1" pad="A"/>
-<contactref element="R31" pad="1"/>
-<wire x1="17.457025" y1="71.628815625" x2="17.457025" y2="74.038815625" width="0.8128" layer="1"/>
-<wire x1="17.457025" y1="74.038815625" x2="17.904525" y2="75.121315625" width="0.8128" layer="1"/>
-</signal>
-<signal name="N$26">
-<contactref element="FD2" pad="A"/>
-<contactref element="R32" pad="1"/>
-<wire x1="17.457025" y1="82.106315625" x2="17.457025" y2="85.151315625" width="0.8128" layer="1"/>
-<wire x1="17.457025" y1="85.151315625" x2="17.904525" y2="85.598815625" width="0.8128" layer="1"/>
-</signal>
-<signal name="N$27">
-<contactref element="FCH" pad="A"/>
-<contactref element="R33" pad="1"/>
-<wire x1="94.559203125" y1="61.51530625" x2="95.688959375" y2="61.51530625" width="0.8128" layer="1"/>
-<wire x1="95.688959375" y1="61.51530625" x2="96.3120625" y2="62.138409375" width="0.8128" layer="1"/>
-<wire x1="96.3120625" y1="62.138409375" x2="96.3120625" y2="63.101309375" width="0.8128" layer="1"/>
-<wire x1="96.3120625" y1="63.101309375" x2="94.63653125" y2="64.776840625" width="0.8128" layer="1"/>
-</signal>
 <signal name="N$30">
