File: Electronics V3/LasaurDriverBoard2.sch (EAGLE design)
At the start: 124 parts, among them IC1 ATMEGA168-20P, IC2 ATMEGA168-20P, IC6 MCP2200SOIC20, Q8 12Mhz, X1 22-23-2021, X3 USB-SMD-NS, Y1 16Mhz, Y2 16Mhz

Commit message: Minor Updates
Minor Updates
Parts:
- removed FCH, FD1, FD2: (no value), led:LED3MM
- removed R31, R32, R33: (no value), resistor:R-EU_M1206
Connections:
- removed net N$25: FD1.A, R31.1
- removed net N$26: FD2.A, R32.1
- removed net N$27: FCH.A, R33.1
- net CHILLER_BIT_SENSE: no longer FCH.C
- net DOOR1: no longer FD1.C
- net DOOR2: no longer FD2.C
- net VCC: no longer R31.2, R32.2, R33.2
Changed lines of the file:
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@@
 <part name="FZP" library="led" deviceset="LED" device="3MM"/>
 <part name="R30" library="resistor" deviceset="R-EU_" device="M1206"/>
-<part name="FD1" library="led" deviceset="LED" device="3MM"/>
-<part name="R31" library="resistor" deviceset="R-EU_" device="M1206"/>
-<part name="FD2" library="led" deviceset="LED" device="3MM"/>
-<part name="R32" library="resistor" deviceset="R-EU_" device="M1206"/>
-<part name="FCH" library="led" deviceset="LED" device="3MM"/>
-<part name="R33" library="resistor" deviceset="R-EU_" device="M1206"/>
 <part name="ZSTEP" library="con-wago-500" deviceset="W237-102" device=""/>
 <part name="ZDIR" library="con-wago-500" deviceset="W237-102" device=""/>
@@
 <instance part="FZP" gate="G$1" x="340.36" y="50.8" rot="R90"/>
 <instance part="R30" gate="G$1" x="332.74" y="50.8" rot="R180"/>
-<instance part="FD1" gate="G$1" x="340.36" y="38.1" rot="R90"/>
-<instance part="R31" gate="G$1" x="332.74" y="38.1" rot="R180"/>
-<instance part="FD2" gate="G$1" x="340.36" y="30.48" rot="R90"/>
-<instance part="R32" gate="G$1" x="332.74" y="30.48" rot="R180"/>
-<instance part="FCH" gate="G$1" x="340.36" y="22.86" rot="R90"/>
-<instance part="R33" gate="G$1" x="332.74" y="22.86" rot="R180"/>
 <instance part="ZSTEP" gate="-1" x="431.8" y="76.2"/>
 <instance part="ZSTEP" gate="-2" x="431.8" y="71.12"/>
@@
 </segment>
 <segment>
-<pinref part="FCH" gate="G$1" pin="C"/>
-<wire x1="345.44" y1="22.86" x2="347.98" y2="22.86" width="0.1524" layer="91"/>
-<label x="337.82" y="22.86" size="1.778" layer="95" font="vector" ratio="10"/>
-</segment>
-<segment>
 <pinref part="IC2" gate="G$1" pin="(PCI21/T1/OC0B)PD5"/>
 <wire x1="581.66" y1="124.46" x2="584.2" y2="124.46" width="0.1524" layer="91"/>
@@
 </segment>
 <segment>
-<pinref part="R31" gate="G$1" pin="2"/>
-<wire x1="327.66" y1="38.1" x2="325.12" y2="38.1" width="0.1524" layer="91"/>
-<label x="320.04" y="38.1" size="1.778" layer="95" font="vector" ratio="10"/>
-</segment>
-<segment>
-<pinref part="R32" gate="G$1" pin="2"/>
-<wire x1="327.66" y1="30.48" x2="325.12" y2="30.48" width="0.1524" layer="91"/>
-<label x="320.04" y="30.48" size="1.778" layer="95" font="vector" ratio="10"/>
-</segment>
-<segment>
-<pinref part="R33" gate="G$1" pin="2"/>
-<wire x1="327.66" y1="22.86" x2="325.12" y2="22.86" width="0.1524" layer="91"/>
-<label x="320.04" y="22.86" size="1.778" layer="95" font="vector" ratio="10"/>
-</segment>
-<segment>
 <wire x1="238.76" y1="38.1" x2="231.14" y2="38.1" width="0.1524" layer="91"/>
 <label x="231.14" y="38.1" size="1.778" layer="95"/>
@@
 <pinref part="DOOR1" gate="-2" pin="KL"/>
 </segment>
-<segment>
-<pinref part="FD1" gate="G$1" pin="C"/>
-<wire x1="345.44" y1="38.1" x2="347.98" y2="38.1" width="0.1524" layer="91"/>
-<label x="347.98" y="38.1" size="1.778" layer="95" font="vector" ratio="10"/>
-</segment>
 </net>
 <net name="DOOR2" class="0">
@@
 <junction x="391.16" y="38.1"/>
 <pinref part="DOOR2" gate="-2" pin="KL"/>
-</segment>
-<segment>
-<pinref part="FD2" gate="G$1" pin="C"/>
-<wire x1="345.44" y1="30.48" x2="347.98" y2="30.48" width="0.1524" layer="91"/>
-<label x="347.98" y="30.48" size="1.778" layer="95" font="vector" ratio="10"/>
 </segment>
 </net>
@@
 </segment>
 </net>
-<net name="N$25" class="0">
-<segment>
-<pinref part="FD1" gate="G$1" pin="A"/>
-<pinref part="R31" gate="G$1" pin="1"/>
-</segment>
-</net>
-<net name="N$26" class="0">
-<segment>
-<pinref part="FD2" gate="G$1" pin="A"/>
-<pinref part="R32" gate="G$1" pin="1"/>
-</segment>
-</net>
-<net name="N$27" class="0">
-<segment>
-<pinref part="FCH" gate="G$1" pin="A"/>
-<pinref part="R33" gate="G$1" pin="1"/>
-</segment>
-</net>
